File: fabMX_keyPad/fabMX_keyPad.kicad_sch (KiCad schematic)
At the start: 114 parts, among them J1 USB_C_Receptacle_USB2.0, J2 Conn_02x03_Odd_Even, J3 Conn_01x04, J6 Conn_01x04, J7 Conn_01x12, SW10 SW_Push, SW11 SW_Push, SW12 SW_Push, SW20 SW_Push, SW21 SW_Push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

Commit message: Fixes from @fkreiner 's feedback at 37C3
Connected NFC_CS' and NFC_RST' signals to MCU
Added additional Jumper-R to connect NFC_3V3 to global 3.3V net
Parts:
- added R18: 0, dipolMods:R_0603_min, symbol Device:R
- R10, R13, R14, R15, R16, R17: now fitted
Connections:
- net A5 is gone; now on net NFC_RST': U1.47 (PB02)
- net D10 is gone; now on net NFC_CS': U1.27 (PA18)
- net 3.3V: now also R18.1
- net NFC_3V3: now also R18.2
Other:
- note added: "A5"
- note added: "D10"
Changed lines of the file:
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@@
     (stroke (width 0) (type default))
   )
-  (wire (pts (xy 186.69 102.87) (xy 196.85 102.87))
+  (wire (pts (xy 184.15 102.87) (xy 196.85 102.87))
     (stroke (width 0) (type default))
   )
@@
     (stroke (width 0) (type default))
   )
-  (wire (pts (xy 186.69 107.95) (xy 196.85 107.95))
+  (wire (pts (xy 184.15 107.95) (xy 196.85 107.95))
     (stroke (width 0) (type default))
   )
@@
     (stroke (width 0) (type default))
   )
-  (wire (pts (xy 186.69 105.41) (xy 196.85 105.41))
+  (wire (pts (xy 184.15 105.41) (xy 196.85 105.41))
     (stroke (width 0) (type default))
   )
@@
     (stroke (width 0) (type default))
   )
-  (wire (pts (xy 186.69 100.33) (xy 196.85 100.33))
+  (wire (pts (xy 251.46 57.15) (xy 254 57.15))
+    (stroke (width 0) (type default))
+  )
+  (wire (pts (xy 184.15 100.33) (xy 196.85 100.33))
     (stroke (width 0) (type default))
   )
@@
     (effects (font (size 1.27 1.27)) (justify left bottom))
   )
+  (text "A5" (at 232.41 64.77 0)
+    (effects (font (size 1.27 1.27)) (justify left bottom))
+  )
   (text "SPI FLASH" (at 162.56 125.73 0)
     (effects (font (size 2.54 2.159) (thickness 0.4318) bold) (justify right bottom))
@@
     (effects (font (size 1.27 1.27)) (justify left bottom))
   )
+  (text "D10" (at 193.04 105.41 0)
+    (effects (font (size 1.27 1.27)) (justify left bottom))
+  )
   (text "NEOPIXEL LED" (at 41.91 125.73 0)
     (effects (font (size 2.54 2.159) (thickness 0.4318) bold) (justify right bottom))
@@
     (effects (font (size 1.27 1.27)) (justify right bottom))
   )
-  (label "A5" (at 243.84 64.77 180) (fields_autoplaced)
-    (effects (font (size 1.27 1.27)) (justify right bottom))
-  )
   (label "SDA" (at 103.505 185.42 0) (fields_autoplaced)
     (effects (font (size 1.27 1.27)) (justify left bottom))
@@
     (effects (font (size 1.2446 1.2446)) (justify left bottom))
   )
-  (label "D13" (at 186.69 102.87 0) (fields_autoplaced)
+  (label "D13" (at 184.15 102.87 0) (fields_autoplaced)
     (effects (font (size 1.27 1.27)) (justify left bottom))
   )
@@
     (effects (font (size 1.27 1.27)) (justify left bottom))
   )
+  (label "NFC_CS'" (at 184.15 105.41 0) (fields_autoplaced)
+    (effects (font (size 1.27 1.27)) (justify left bottom))
+  )
   (label "MISO" (at 186.69 90.17 0) (fields_autoplaced)
     (effects (font (size 1.27 1.27)) (justify left bottom))
   )
+  (label "NFC_RST'" (at 243.84 64.77 180) (fields_autoplaced)
+    (effects (font (size 1.27 1.27)) (justify right bottom))
+  )
   (label "SCL" (at 261.62 27.94 0) (fields_autoplaced)
     (effects (font (size 1.27 1.27)) (justify left bottom))
@@
     (effects (font (size 1.27 1.27)) (justify left bottom))
   )
-  (label "ROW3" (at 186.69 100.33 0) (fields_autoplaced)
+  (label "ROW3" (at 184.15 100.33 0) (fields_autoplaced)
     (effects (font (size 1.27 1.27)) (justify left bottom))
   )
@@
     (effects (font (size 1.2446 1.2446)) (justify left bottom))
   )
-  (label "D12" (at 186.69 107.95 0) (fields_autoplaced)
+  (label "D12" (at 184.15 107.95 0) (fields_autoplaced)
     (effects (font (size 1.27 1.27)) (justify left bottom))
   )
@@
     (effects (font (size 1.27 1.27)) (justify left bottom))
   )
-  (label "D10" (at 186.69 105.41 0) (fields_autoplaced)
-    (effects (font (size 1.27 1.27)) (justify left bottom))
-  )
   (label "ROW3" (at 73.66 102.87 0) (fields_autoplaced)
     (effects (font (size 1.27 1.27)) (justify left bottom))
@@
     )
   )
+  (symbol (lib_id "Device:R") (at 257.81 57.15 90) (unit 1)
+    (in_bom yes) (on_board yes) (dnp no)
+    (property "Reference" "R18" (at 257.81 57.15 90)
+      (effects (font (size 1.27 1.27)))
+    )
+    (property "Value" "0" (at 256.54 54.61 90)
+      (effects (font (size 1.27 1.27)) hide)
+    )
+    (property "Footprint" "dipolMods:R_0603_min" (at 257.81 58.928 90)
+      (effects (font (size 1.27 1.27)) hide)
+    )
+    (property "Datasheet" "~" (at 257.81 57.15 0)
+      (effects (font (size 1.27 1.27)) hide)
+    )
+    (pin "1")
+    (pin "2")
+    (instances
+      (project "fabMX_keyPad"
+        (path "/273c846b-2489-4e3b-aca6-4c67ab5363d9"
+          (reference "R18") (unit 1)
+        )
+      )
+    )
+  )
   (symbol (lib_id "Switch:SW_Push") (at 86.36 95.25 0) (unit 1)
     (in_bom yes) (on_board yes) (dnp no) (fields_autoplaced)
@@
   )
   (symbol (lib_id "Device:R") (at 257.81 49.53 90) (unit 1)
-    (in_bom yes) (on_board yes) (dnp yes)
+    (in_bom yes) (on_board yes) (dnp no)
     (property "Reference" "R16" (at 257.81 49.53 90)
       (effects (font (size 1.27 1.27)))
@@
     )
   )
+  (symbol (lib_id "miniMetro-eagle-import:3.3V") (at 248.92 57.15 90) (unit 1)
+    (in_bom yes) (on_board yes) (dnp no)
+    (property "Reference" "#017" (at 248.92 57.15 0)
+      (effects (font (size 1.27 1.27)) hide)
+    )
+    (property "Value" "3.3V" (at 248.92 57.15 90)
+      (effects (font (size 1.27 1.0795)) (justify left))
+    )
+    (property "Footprint" "" (at 248.92 57.15 0)
+      (effects (font (size 1.27 1.27)) hide)
+    )
+    (property "Datasheet" "" (at 248.92 57.15 0)
+      (effects (font (size 1.27 1.27)) hide)
+    )
+    (pin "1")
+    (instances
+      (project "fabMX_keyPad"
+        (path "/273c846b-2489-4e3b-aca6-4c67ab5363d9"
+          (reference "#017") (unit 1)
+        )
+      )
+    )
+  )
   (symbol (lib_id "CostumLibary:WS2812B") (at 151.13 106.68 0) (unit 1)
     (in_bom yes) (on_board yes) (dnp no)
@@
   )
   (symbol (lib_id "Device:R") (at 257.81 46.99 90) (unit 1)
-    (in_bom yes) (on_board yes) (dnp yes)
+    (in_bom yes) (on_board yes) (dnp no)
     (property "Reference" "R15" (at 257.81 46.99 90)
       (effects (font (size 1.27 1.27)))
@@
   )
   (symbol (lib_id "Device:R") (at 257.81 44.45 90) (unit 1)
-    (in_bom yes) (on_board yes) (dnp yes)
+    (in_bom yes) (on_board yes) (dnp no)
     (property "Reference" "R14" (at 257.81 44.45 90)
       (effects (font (size 1.27 1.27)))
@@
   )
   (symbol (lib_id "Device:R") (at 257.81 41.91 90) (unit 1)
-    (in_bom yes) (on_board yes) (dnp yes)
+    (in_bom yes) (on_board yes) (dnp no)
     (property "Reference" "R13" (at 257.81 41.91 90)
       (effects (font (size 1.27 1.27)))
@@
   )
   (symbol (lib_id "Device:R") (at 257.81 39.37 90) (unit 1)
-    (in_bom yes) (on_board yes) (dnp yes)
+    (in_bom yes) (on_board yes) (dnp no)
     (property "Reference" "R10" (at 257.81 39.37 90)
       (effects (font (size 1.27 1.27)))
@@
   )
   (symbol (lib_id "Device:R") (at 257.81 54.61 90) (unit 1)
-    (in_bom yes) (on_board yes) (dnp yes)
+    (in_bom yes) (on_board yes) (dnp no)
     (property "Reference" "R17" (at 257.81 54.61 90)
       (effects (font (size 1.27 1.27)))

Commit message: some Work on BOM
work not yet finished...wait for more updates before odering please
Parts:
- C1, C12, C13, C14, C15, C2, C3, C9: BOM comment (none) -> generic MLCC - Sortiment?; Mnf (none) -> GENERIC
- C10, C11, C16, C17, C18, C19, C20, C21, C22, C23, C24, C25, C4, C5, C6, C7, C8: value 100n -> 100nF 25V X7R; BOM comment (none) -> generic MLCC - Sortiment?; Mnf (none) -> GENERIC
- D10, D11, D12, D20, D21, D22, D30, D31, D32, DO0, DO1, DO2: ALT1 LCSC# (none) -> C181134; BOM comment (none) -> -; Mnf (none) -> GENERIC; Mnf# (none) -> diverse
- D2, LED10, LED11, LED12, LED20, LED21, LED22, LED30, LED31, LED32, LEDO0, LEDO1, LEDO2: BOM comment (none) -> AL hätte noch welche
- F1: ALT1 LCSC# (none) -> 0R R 0603; BOM comment (none) -> 0R 0603 could be used; Digikey# (none) -> F5759CT-ND; Mouser# (none) -> 576-0402L050SLKR
- FB1: ALT1 LCSC# (none) -> 0R 0603; BOM comment (none) -> 0R 0603 could be used; Mnf (none) -> GENERIC
- H1, H2: BOM comment (none) -> no part, jus holes in PCB; Mnf (none) -> no BOM; now left out of the parts list
- H3, H4, H5: BOM comment (none) -> no part, jus holes in PCB; Mnf (none) -> no BOM
- J1: BOM comment (none) -> standard USB-C USB2.0 connector - dev/debug only; Digikey# (none) -> 2073-USB4105-GF-ACT-ND; LCSC# (none) -> C2988369; Mnf (none) -> GENERIC; Mnf# (none) -> diverse; Mouser# (none) -> 640-USB4105-GF-A
- J2: BOM comment (none) -> no Part, just Pads; Mnf (none) -> no BOM; now left out of the parts list
- J3: BOM comment (none) -> optional - QWIC connector; Digikey# (none) -> 455-SM04B-SRSS-TBCT-ND; Farnell# (none) -> 1830839; Mnf (none) -> JST; Mnf# (none) -> SM04B-SRSS-TB
- J6: Mnf (none) -> GENERIC
- J7: BOM comment (none) -> oder nur anlöten???
- JP1: BOM comment (none) -> no Part, just Pads; Mnf (none) -> GENERIC
- LED1, LED_RX1, LED_TX1, ON1: BOM comment (none) -> optional/debug - generic SMD LED; Mnf (none) -> GENERIC
- R1, R10, R11, R12, R13, R14, R15, R16, R17, R18, R2, R3, R4, R5, R6, R7, R8, R9: BOM comment (none) -> generic R0603; Mnf (none) -> GENERIC
- SW10, SW11, SW12, SW20, SW21, SW22, SW30, SW31, SW32, SWO0, SWO1, SWO2: BOM comment (none) -> cherry-style key switch
- TP1, TP10, TP11, TP12, TP2, TP3, TP4, TP5, TP6, TP7, TP8, TP9: BOM comment (none) -> no Part, just Pads; Mnf (none) -> no BOM
- U1: BOM comment (none) -> -; LCSC# (none) -> C614475; Mnf (none) -> Microchip; Mouser# (none) -> 556-ATSAMD21G18A-MUT; Part# (none) -> ATSAMD21G18A-M*
- U2: BOM comment (none) -> optional - not need in first iteration; now not fitted
- X1: BOM comment (none) -> je nach Montage etwas flexibel zu bestücken - aus Bestand?; Mnf MISC/VORRAT -> GENERIC

Commit message: BOM update + move to kicad8
Parts:
- C1, C2: now not fitted
- D10, D11, D12, D20, D21, D22, D30, D31, D32, DO0, DO1, DO2: Digikey# (none) -> 4878-1N4148WCT-ND
- D2, LED10, LED11, LED12, LED20, LED21, LED22, LED30, LED31, LED32, LEDO0, LEDO1, LEDO2: Digikey# (none) -> 1528-4492-ND; Mnf# (none) -> diverse
- D3: Digikey# (none) -> 4878-SL1MCT-ND
- J6: Farnell# (none) -> 3817900; Mnf GENERIC -> WE/Generic; Mnf# (none) -> 61000413321; now not fitted
- U1: Digikey# (none) -> ATSAMD21G18A-MUTCT-ND
- U4: Digikey# (none) -> AP2112K-3.3TRG1DICT-ND
- Y1: BOM comment (none) -> DNP; now not fitted
